File: KiCAD/FWS_20A/FWS_20A.kicad_pcb (KiCad board)
At the start: 2 copper layers, 75 parts, among them J1 pwr, J3 Conn_01x09_Socket, J4 Conn_01x03_Pin, J5 sense, Q1 DMN32D2LDF, Q2 BC846, Q6 DMN32D2LDF, U1 XMSM0L1306SRGER, U12 ADS1015IDGS, U2 FDMS8333L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

Commit message: asd
Parts:
- removed Q2: BC846, Package_TO_SOT_SMD:SOT-23
- removed R18, R24, R25: 750, Resistor_SMD:R_1206_3216Metric_Pad1.30x1.75mm_HandSolder
- removed R22: 4.99k, Resistor_SMD:R_1206_3216Metric_Pad1.30x1.75mm_HandSolder
- added J2: Conn_01x02_Pin, Connector_PinHeader_2.54mm:PinHeader_1x02_P2.54mm_Vertical, F.Cu at (112.2, 68.7)
- added R13: 2.49k, Resistor_SMD:R_0603_1608Metric, F.Cu at (129.8, 61.0)
- added SW2: SW_Push, Button_Switch_SMD:SW_SPST_PTS645Sx43SMTR92, F.Cu at (156.4, 68.0)
- added U11: FCX495, Package_TO_SOT_SMD:SOT-89-3, F.Cu at (111.8, 56.2)
- C2, C7: footprint Capacitor_THT:C_Radial_D6.3mm_H11.0mm_P2.50mm -> Capacitor_THT:CP_Radial_D6.3mm_P2.50mm
- D6, D7: moved to B.Cu
- J1: footprint Connector_Wago:Wago_734-134_1x04_P3.50mm_Vertical -> Connector_Wire:SolderWire-0.75sqmm_1x04_P4.8mm_D1.25mm_OD2.3mm
- J4: value Conn_01x03_Pin -> Conn_01x02_Pin; footprint Connector_PinHeader_2.54mm:PinHeader_1x03_P2.54mm_Vertical -> Connector_PinHeader_2.54mm:PinHeader_1x02_P2.54mm_Vertical
- R1, R5: value 8.2 -> 49.9k; footprint Resistor_SMD:R_2816_7142Metric_Pad3.20x4.45mm_HandSolder -> Resistor_SMD:R_1206_3216Metric_Pad1.30x1.75mm_HandSolder
- R16: value 750 -> 2.49k; footprint Resistor_SMD:R_1206_3216Metric_Pad1.30x1.75mm_HandSolder -> Resistor_SMD:R_0603_1608Metric
- R17, R9: value 150 -> 2.49k; footprint Resistor_SMD:R_1206_3216Metric_Pad1.30x1.75mm_HandSolder -> Resistor_SMD:R_0603_1608Metric
- R2, R6: value 8.2 -> 5.1; footprint Resistor_SMD:R_2816_7142Metric_Pad3.20x4.45mm_HandSolder -> Resistor_SMD:R_1206_3216Metric_Pad1.30x1.75mm_HandSolder
- R21: value 4.99k -> 2.49k; footprint Resistor_SMD:R_1206_3216Metric_Pad1.30x1.75mm_HandSolder -> Resistor_SMD:R_0603_1608Metric
- R3, R4, R7, R8: footprint Resistor_SMD:R_2512_6332Metric_Pad1.40x3.35mm_HandSolder -> Resistor_SMD:R_1206_3216Metric_Pad1.30x1.75mm_HandSolder
- moved R11 146.2 mm to (194.0, 70.2)
- moved R19 141.7 mm to (194.0, 80.1)
- moved R21 141.0 mm to (194.0, 83.4)
- moved D11 137.4 mm to (199.0, 69.8)
- moved D14 137.4 mm to (199.0, 77.6)
- moved D16 137.4 mm to (199.0, 80.2)
- moved R20 102.1 mm to (153.8, 80.2)
- moved J3 90.0 mm to (142.2, 89.2), turned to 180 degrees
- moved Q6 89.6 mm to (135.0, 61.6), turned to 180 degrees
- moved U2 84.3 mm to (132.6, 34.2), turned to 90 degrees
- moved U3 83.1 mm to (132.6, 45.6), turned to 90 degrees
- moved R9 82.2 mm to (129.8, 57.8), turned to -90 degrees
- moved C2 80.4 mm to (140.8, 44.7), turned to 180 degrees
- moved U7 79.7 mm to (122.0, 34.2), turned to 90 degrees
- moved R14 79.2 mm to (128.0, 65.6), turned to 180 degrees
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Connections:
- C11 pad 1: Net-(J4-Pin_3) -> Net-(J2-Pin_2)
- D3 pad 2: Net-(D3-A) -> +BATT
- J1 pad 1: /M- -> +BATT
- J1 pad 3: GND -> /M-
- J1 pad 4: Net-(D3-A) -> GND
- R1 pad 1: Net-(D2-A) -> /S_Front
- R1 pad 2: +12V -> Net-(U12-AIN1)
- R16 pad 1: Net-(D12-A) -> Net-(D13-A)
- R16 pad 2: +3V3 -> +12V
- R17 pad 1: /S_Front -> Net-(D12-A)
- R17 pad 2: Net-(U12-AIN1) -> +12V
- R4 pad 1: Net-(D5-K) -> Net-(D5-A)
- R4 pad 2: Net-(D5-A) -> Net-(D5-K)
- R5 pad 1: Net-(D8-A) -> Net-(U12-AIN2)
- R5 pad 2: +12V -> /S_Feedback
- R8 pad 1: Net-(D10-K) -> Net-(D10-A)
- R8 pad 2: Net-(D10-A) -> Net-(D10-K)
- R9 pad 1: Net-(U12-AIN2) -> Net-(D19-A)
- R9 pad 2: /S_Feedback -> +12V
- U2 pad 3: +12V -> +BATT
- U4 pad 2: /TIMG2_C0 -> /TIMG2_C1
- U4 pad 3: /TIMG2_C1 -> /TIMG2_C0
- U5 pad 2: /TIMG4_C0 -> /TIMG4_C1
- U5 pad 3: /TIMG4_C1 -> /TIMG4_C0
- U6 pad 1: Net-(J4-Pin_3) -> Net-(J2-Pin_2)
- U7 pad 3: +12V -> +BATT
Routing:
- net Net-(D3-K): track 0.00 -> 26.4 mm, vias 0 -> 2
- net +3V3: track 0.00 -> 23.3 mm
- net /TIMG4_C0: track 0.00 -> 20.5 mm, vias 0 -> 2
- net Net-(D9-K): track 0.00 -> 19.6 mm
- net /TIMG4_C1: track 0.00 -> 19.0 mm, vias 0 -> 2
- net /M+: track 0.00 -> 18.1 mm, vias 0 -> 4
- net Net-(D8-K): track 0.00 -> 18.0 mm
- net +12V: track 0.00 -> 17.9 mm
- net Net-(D4-K): track 0.00 -> 17.8 mm
- net /M-: track 0.00 -> 16.4 mm, vias 0 -> 7
- net /TIMG2_C0: track 0.00 -> 14.4 mm, vias 0 -> 2
- net /XDS_RESET_OUT: track 0.00 -> 14.3 mm
- net /TIMG2_C1: track 0.00 -> 14.3 mm
- net Net-(D10-A): track 0.00 -> 13.2 mm, vias 0 -> 3
- net Net-(D2-K): track 0.00 -> 12.0 mm, vias 0 -> 1
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- added copper zone on F.Cu, net +12V
- added copper zone on F.Cu, net +BATT
- added copper zone on B.Cu, net /M+
- added copper zone on F.Cu, net /M+
- added copper zone on B.Cu, net /M-
- added copper zone on F.Cu, net /M-
- added copper zone on B.Cu, net GND
- added copper zone on F.Cu, net GND
Other:
- board outline added: 36.6 x 65 mm
- board text added: "TIMG2_C0"
- board text added: "TIMG2_C1"
- board text added: "TIMG4_C0"
- board text added: "TIMG4_C1"

Commit message: thanks random guy that slaved away at the lower layout
Parts:
- moved D11 67.7 mm to (132.8, 83.8), turned to 90 degrees
- moved R11 65.6 mm to (128.8, 77.4), turned to 90 degrees
- moved D16 64.1 mm to (135.0, 83.8), turned to 90 degrees
- moved R21 64.0 mm to (131.0, 72.0), turned to 90 degrees
- moved D14 61.7 mm to (137.6, 83.8), turned to 90 degrees
- moved TP1 61.4 mm to (129.8, 89.6)
- moved R19 60.1 mm to (134.4, 72.2), turned to 180 degrees
- moved TP2 57.9 mm to (125.0, 89.8)
- moved R50 31.9 mm to (121.4, 68.2), turned to 90 degrees
- moved R12 29.3 mm to (124.2, 68.2), turned to 90 degrees
- moved R20 26.3 mm to (128.8, 72.0), turned to -90 degrees
- moved R5 23.4 mm to (123.8, 77.4), turned to -90 degrees
- moved SW2 23.1 mm to (135.2, 77.2)
- moved C13 21.7 mm to (126.2, 77.4), turned to -90 degrees
- moved R23 21.0 mm to (117.4, 76.2), turned to 180 degrees
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Connections:
- J5 pad 4: +3V3 -> Net-(J5-Pin_4)
- J5 pad 6: Net-(J5-Pin_6) -> +3V3
- TP2 pad 1: Net-(J5-Pin_6) -> Net-(J5-Pin_4)
Routing:
- net +3V3: track 23.3 -> 96.7 mm, vias 0 -> 4
- net /PA24: track 0.00 -> 32.9 mm, vias 0 -> 2
- net +12V: track 17.9 -> 39.2 mm, vias 0 -> 2
- net /S_Feedback: track 0.00 -> 17.9 mm
- net /XDS_TARG_RXD: track 0.00 -> 17.6 mm
- net /XDS_TARG_TXD: track 0.00 -> 15.5 mm, vias 0 -> 1
- net /XDS_TMS_SWDIO: track 0.00 -> 14.7 mm, vias 0 -> 1
- net /XDS_RESET_OUT: track 14.3 -> 28.3 mm, vias 0 -> 2
- net /XDS_BSL_INVOKE: track 0.00 -> 13.0 mm, vias 0 -> 1
- net /XDS_TCK_SWDCLK: track 0.00 -> 12.4 mm, vias 0 -> 1
- net Net-(D16-A): track 0.00 -> 11.8 mm
- net Net-(D14-A): track 0.00 -> 11.5 mm
- net Net-(J5-Pin_5): track 0.00 -> 10.5 mm
- net Net-(U12-AIN0): track 0.00 -> 9.91 mm, vias 0 -> 1
- net /S_Front: track 0.00 -> 8.38 mm
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Other:
- board text added: "I'm sorry George and Grant"

Commit message: asd
Parts:
- added R18: 4.99k, Resistor_SMD:R_1206_3216Metric_Pad1.30x1.75mm_HandSolder, F.Cu at (125.9, 85.4)
- moved TP3 1.40 mm to (112.2, 75.0)
Connections:
- J5 pad 6: +3V3 -> /Sensor Bias
Routing:
- net +3V3: track 96.7 -> 87.1 mm
- net /Sensor Bias: track 0.00 -> 4.71 mm
- net Net-(U12-AIN0): track 9.91 -> 10.5 mm
Other:
- board text added: "12V"
- board text added: "3.3V"
- board text added: "3v3 OUT"
- board text added: "3v3 join board <-> XDS"
- board text added: "Front Angle"
- board text added: "GND"
- board text added: "LV+ (~12V)"
- board text added: "M+"
- board text added: "M-"
- board text added: "Rear Angle"
- board text added: "onboard 3v3 rail <-> PSU"
- board text added: "sensors"
- board text added: "unused A"
- board text added: "unused B"

Commit message: sad
Parts:
- added TP4: TestPoint, TestPoint:TestPoint_Pad_D2.0mm, B.Cu at (123.8, 70.2)
- added TP5: TestPoint, TestPoint:TestPoint_Pad_D2.0mm, B.Cu at (126.2, 73.8)
Routing:
- net /I2C0_SCL: track 11.3 -> 14.0 mm, vias 0 -> 1
- net /I2C0_SDA: track 10.2 -> 13.0 mm, vias 0 -> 1
Other:
- board text added: "ADC SCL"
- board text added: "ADC SDA"
- board text added: "ADC: ADS1015IDGS"

Commit message: cleaned a bit
Parts:
- added D15: 3.3V, Diode_SMD:D_SOD-323, B.Cu at (121.0, 77.4)
- added D17: 3.3V, Diode_SMD:D_SOD-323, B.Cu at (123.8, 77.4)
- added TP6: TestPoint, TestPoint:TestPoint_Pad_D2.0mm, B.Cu at (135.8, 63.0)
- added TP7: TestPoint, TestPoint:TestPoint_Pad_D2.0mm, B.Cu at (138.9, 63.5)
- added TP8: TestPoint, TestPoint:TestPoint_Pad_D2.0mm, B.Cu at (126.3, 62.8)
- added TP9: TestPoint, TestPoint:TestPoint_Pad_D2.0mm, B.Cu at (123.6, 64.1)
- moved TP4 2.21 mm to (126.0, 70.0)
- moved TP5 1.84 mm to (127.6, 72.6)
Routing:
- net /I2C0_SCL: track 14.0 -> 11.3 mm
- net /I2C0_SDA: track 13.0 -> 10.2 mm
- net /TIMG4_C0: track 20.5 -> 23.2 mm
- net Net-(D15-K): track 5.67 -> 6.17 mm, vias 0 -> 1
- net /TIMG2_C1: vias 0 -> 1
- net Net-(D17-K): vias 0 -> 1
- net GND: vias 52 -> 55
- net /TIMG2_C0: vias 2 -> 3
Other:
- board text added: "3v3 out"
- board text added: "5v out"
- board text added: "A HI"
- board text added: "A LO"
- board text added: "B HI"
- board text added: "B LO"
- board text added: "BSL"
- board text added: "RESET"
- board text added: "SWDCLK"
- board text added: "SWDIO"
- board text added: "TARG_RX"
- board text added: "TARG_TX"
- board text added: "github.com/gregclacker/FourWheelSteering v1"

Commit message: more silkscreen txt
Parts:
- added H1: MountingHole, MountingHole:MountingHole_2.2mm_M2_DIN965, F.Cu at (121.5, 92.6)
- added H2: MountingHole, MountingHole:MountingHole_2.2mm_M2_DIN965, F.Cu at (110.6, 32.7)
Routing:
- net GND: vias 55 -> 61
Other:
- board text added: "unused ADC CH0"

Commit message: cleaned up a bit
Parts:
- removed R18, R23, R50: 4.99k, Resistor_SMD:R_1206_3216Metric_Pad1.30x1.75mm_HandSolder
- removed TP3: TestPoint, TestPoint:TestPoint_Loop_D2.50mm_Drill1.0mm_LowProfile
- removed TP4, TP5, TP6, TP7, TP8, TP9: TestPoint, TestPoint:TestPoint_Pad_D2.0mm
- added C10: 10u, Capacitor_SMD:C_1206_3216Metric_Pad1.33x1.80mm_HandSolder, F.Cu at (158.7, 68.0)
- added C16: 220n, Capacitor_SMD:C_1206_3216Metric_Pad1.33x1.80mm_HandSolder, F.Cu at (172.8, 47.8)
- added C17: 10u, Capacitor_SMD:C_1206_3216Metric_Pad1.33x1.80mm_HandSolder, F.Cu at (172.8, 51.2)
- added C18: 220n, Capacitor_SMD:C_1206_3216Metric_Pad1.33x1.80mm_HandSolder, F.Cu at (172.8, 54.5)
- added C19: 220n, Capacitor_SMD:C_1206_3216Metric_Pad1.33x1.80mm_HandSolder, F.Cu at (158.7, 71.3)
- added C20: 220n, Capacitor_SMD:C_1206_3216Metric_Pad1.33x1.80mm_HandSolder, F.Cu at (158.7, 74.7)
- added H3: MountingHole, MountingHole:MountingHole_2.2mm_M2_DIN965, F.Cu at (183.6, 64.2)
- added J16: USB_B_Micro, Connector_USB:USB_Micro-B_Amphenol_10118194-0001LF_Horizontal, F.Cu at (160.8, 61.3)
- added J6: USB_B_Micro, Connector_USB:USB_Micro-B_Amphenol_10118194-0001LF_Horizontal, F.Cu at (160.8, 41.2)
- added R22: 49.9k, Resistor_SMD:R_1206_3216Metric_Pad1.30x1.75mm_HandSolder, F.Cu at (183.9, 59.9)
- added U10: MCP3421A0T-ECH, Package_TO_SOT_SMD:SOT-23-6, F.Cu at (178.3, 65.2)
- added U13: ISO7721D, Package_SO:SOIC-8_3.9x4.9mm_P1.27mm, F.Cu at (166.0, 69.7)
- added U14: L78L05_SOT89, Package_TO_SOT_SMD:SOT-89-3, F.Cu at (167.1, 49.3)
- added U15: FT230XS, Package_SO:SSOP-16_3.9x4.9mm_P0.635mm, F.Cu at (159.7, 49.8)
- added U16: ISO7721D, Package_SO:SOIC-8_3.9x4.9mm_P1.27mm, F.Cu at (170.1, 41.4)
- added U17: FT230XS, Package_SO:SSOP-16_3.9x4.9mm_P0.635mm, F.Cu at (169.8, 61.8)
- added U9: MCP3421A0T-ECH, Package_TO_SOT_SMD:SOT-23-6, F.Cu at (178.3, 60.6)
- D15, D17: value 3.3V -> BAT54S; footprint Diode_SMD:D_SOD-323 -> Package_TO_SOT_SMD:SOT-23-3
- R5: value 49.9k -> 200k; footprint Resistor_SMD:R_1206_3216Metric_Pad1.30x1.75mm_HandSolder -> Resistor_SMD:R_0805_2012Metric_Pad1.20x1.40mm_HandSolder
- U12: value ADS1015IDGS -> L78L05_SOT89; footprint Package_SO:TSSOP-10_3x3mm_P0.5mm -> Package_TO_SOT_SMD:SOT-89-3
Connections:
- C12 pad 1: Net-(D15-K) -> Net-(U12-OUT)
- C12 pad 2: GND -> /isolated TTL/GND
- C13 pad 1: Net-(D17-K) -> Net-(J6-VBUS)
- C13 pad 2: GND -> /isolated TTL1/GND
- D15 pad 1: Net-(D15-K) -> GND
- D15 pad 2: GND -> +3V3
- D17 pad 1: Net-(D17-K) -> GND
- D17 pad 2: GND -> +3V3
- J5 pad 6: /Sensor Bias -> /Sensor_Supply
- R1 pad 1: /S_Front -> Net-(D15-COM)
- R1 pad 2: Net-(D15-K) -> Net-(R1-Pad2)
- R10 pad 1: Net-(D1-K) -> Net-(R1-Pad2)
- R10 pad 2: Net-(D3-K) -> /S_Feedback
- R12 pad 1: Net-(U12-AIN3) -> Net-(R12-Pad1)
- R12 pad 2: +12V -> /S_Front
- R5 pad 1: Net-(D17-K) -> Net-(D1-K)
- R5 pad 2: /S_Feedback -> Net-(D3-K)
- U12 pad 1: GND -> Net-(U12-OUT)
- U12 pad 2: /PA24 -> /isolated TTL/GND
- U12 pad 3: GND -> Net-(J16-VBUS)
Routing:
- net /Sensor_Supply: track 0.00 -> 4.71 mm
- net /Sensor Bias: track 4.71 -> 0.00 mm
