File: KiCAD/FWS_20A/FWS_20A.kicad_sch (KiCad schematic)
At the start: 14 parts, among them J1 sense, J2 pwr, Q2 BC846, U1 XMSM0L1306SRGER, U2 FDMS8333L, U3 FDMS8333L, U4 LM5109BSD, U6 L78L33_SO8

Commit message: maybe schematic
Parts:
- removed J2: pwr, symbol Connector:Conn_01x04_Pin
- removed R27: 100k, Resistor_SMD:R_1206_3216Metric_Pad1.30x1.75mm_HandSolder, symbol Device:R_US
- added C12, C13, C15, C4, C5, C9: 220n, Capacitor_SMD:C_1206_3216Metric_Pad1.33x1.80mm_HandSolder, symbol Device:C_Small
- added C2, C7: 44uF 63V, Capacitor_THT:C_Radial_D6.3mm_H11.0mm_P2.50mm, symbol Device:C_Polarized_Small_US
- added C3, C6: 22u, Capacitor_SMD:C_1206_3216Metric_Pad1.33x1.80mm_HandSolder, symbol Device:C_Small
- added C8: 10u, Capacitor_SMD:C_1206_3216Metric_Pad1.33x1.80mm_HandSolder, symbol Device:C_Small
- added D10, D2, D4, D5, D8, D9: 100V 3A, FWS_footprints:PMDE, symbol Device:D_Schottky_Small
- added D11, D12, D13, D14, D16, D18, D19: LED, LED_SMD:LED_0603_1608Metric, symbol Device:LED
- added D6, D7: 39V 10W, Diode_SMD:D_SMC_Handsoldering, symbol Device:D_Zener_Small
- added J3: Conn_01x09_Socket, Connector_PinHeader_2.54mm:PinHeader_1x09_P2.54mm_Vertical, symbol Connector:Conn_01x09_Socket
- added J4: Conn_01x03_Pin, Connector_PinHeader_2.54mm:PinHeader_1x03_P2.54mm_Vertical, symbol Connector:Conn_01x03_Pin
- added J5: sense, Connector_Molex:Molex_Micro-Fit_3.0_43045-0600_2x03_P3.00mm_Horizontal, symbol Connector:Conn_01x06_Pin
- added Q1, Q6: DMN32D2LDF, Package_TO_SOT_SMD:SOT-353_SC-70-5, symbol Transistor_FET:DMN32D2LDF
- added R1, R2, R5, R6: 8.2, Resistor_SMD:R_2816_7142Metric_Pad3.20x4.45mm_HandSolder, symbol Device:R_Small_US
- added R10, R12, R20: 49.9k, Resistor_SMD:R_1206_3216Metric_Pad1.30x1.75mm_HandSolder, symbol Device:R_US
- added R11, R16, R18, R19, R24, R25: 750, Resistor_SMD:R_1206_3216Metric_Pad1.30x1.75mm_HandSolder, symbol Device:R_US
- added R14, R15, R21, R22, R23, R50: 4.99k, Resistor_SMD:R_1206_3216Metric_Pad1.30x1.75mm_HandSolder, symbol Device:R_US
- added R17, R9: 150, Resistor_SMD:R_1206_3216Metric_Pad1.30x1.75mm_HandSolder, symbol Device:R_US
- added R3, R4, R7, R8: 5.1, Resistor_SMD:R_2512_6332Metric_Pad1.40x3.35mm_HandSolder, symbol Device:R_Small_US
- added SW2: SW_Push, Button_Switch_SMD:SW_SPST_PTS645Sx43SMTR92, symbol Switch:SW_Push
- added TP1, TP2, TP3: TestPoint, TestPoint:TestPoint_Loop_D2.50mm_Drill1.0mm_LowProfile, symbol Connector:TestPoint
- added U12: ADS1015IDGS, Package_SO:TSSOP-10_3x3mm_P0.5mm, symbol Analog_ADC:ADS1015IDGS
- added U5: LM5109BSD, Package_SON:WSON-8-1EP_4x4mm_P0.8mm_EP2.6x3mm, symbol Driver_FET:LM5109BSD
- added U7, U8: FDMS8333L, FWS_footprints:Power 56, symbol FWS_symbols:FDMS8333L
- J1: value sense -> pwr; footprint (none) -> Connector_Wago:Wago_734-134_1x04_P3.50mm_Vertical
- U1: mouser (none) -> https://www.mouser.com/ProductDetail/Texas-Instruments/MSPM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
Connections:
- net +12V: now also C14.1, C3.2, C4.1, C5.1, C6.2, R1.2, R12.2, R2.2, R21.2, R22.1, R5.2, R6.2, U5.1 (VDD), U7.3 (D); no longer C11.1
- net +3V3: now also U1.3 (VDD), C8.1, C9.2, J4.2 (Pin_2), J5.4 (Pin_4), R11.2, R14.2, R15.1, R16.2, R18.2, R20.1, R23.2, R24.2, R25.2, U12.8 (VDD); no longer C14.1, U6.1 (OUT)
- net GND: now also J1.3 (Pin_3), U1.25 (VSS), U1.4 (VSS), C12.2, C13.2, C15.2, C3.1, C4.2, C5.2, C6.1, C8.2, C9.1, D11.1 (K), D14.1 (K), D16.1 (K), J3.1 (Pin_1), J5.3 (Pin_3), Q1.2 (S), Q6.2 (S), R50.2, SW2.2, U12.1 (ADDR), U12.3 (GND), U5.4 (VSS), U5.9 (VSS), U8.1 (S)
- net M+: now also J1.2 (Pin_2), C2.2, D6.1 (K), D7.2 (A)
- net M-: now also J1.1 (Pin_1), C7.2, D6.2 (A), D7.1 (K), U5.6 (HS), U7.1 (S), U8.3 (D)
- net at C1.1, D1.1 (K), Q2.1 (B): now also R10.1
- net at D3.1 (K), Q2.3 (C): now also R10.2
- net at D3.2 (A): now also J1.4 (Pin_4)
- net at U2.2 (G): now also D4.2 (A), R3.2; no longer U4.7 (HO)
- net TIMG4_C1: now reaches U1.10 (PA11)
- net TIMG4_C1: now also Q1.3 (G2), U5.3 (LI)
- net I2C0_SCL: now reaches U1.11 (PA15/A9)
- net I2C0_SCL: now also R14.1, U12.10 (SCL)
- net I2C0_SDA: now reaches U1.12 (PA16/A8)
- net I2C0_SDA: now also R15.2, U12.9 (SDA)
- net XDS_BSL_INVOKE: now reaches U1.14 (PA18/A7)
- net XDS_BSL_INVOKE: now also J3.9 (Pin_9)
- net XDS_TMS_SWDIO: now reaches U1.15 (PA19/SWDIO)
- net XDS_TMS_SWDIO: now also J3.7 (Pin_7)
- net XDS_TCK_SWDCLK: now reaches U1.16 (PA20/A6/SWCLK)
- net XDS_TCK_SWDCLK: now also J3.8 (Pin_8)
- net PA22: now reaches U1.18 (PA22/A4)
- net PA22: now also R19.2
- net XDS_RESET_OUT: now reaches U1.2 (NRST)
- net XDS_RESET_OUT: now also J3.6 (Pin_6), R20.2, SW2.1
- net PA24: now reaches U1.20 (PA24/A3)
- net PA24: now also R23.1, U12.2 (ALERT/RDY)
- net XDS_TARG_TXD: now reaches U1.21 (PA25/A2)
- net XDS_TARG_TXD: now also J3.5 (Pin_5)
- net XDS_TARG_RXD: now reaches U1.22 (PA26/A1)
- net XDS_TARG_RXD: now also J3.4 (Pin_4)
- net at U1.23 (VCORE): now also C15.1
- net TIMG2_C0: now reaches U1.6 (PA3)
- net TIMG2_C0: now also U4.2 (HI), Q6.1 (G1)
- net TIMG2_C1: now reaches U1.7 (PA4)
- net TIMG2_C1: now also U4.3 (LI), Q6.3 (G2)
- net TIMG4_C0: now reaches U1.9 (PA10)
- net TIMG4_C0: now also Q1.1 (G1), U5.2 (HI)
- net at U4.5 (LO): now also D5.1 (K), R4.1; no longer U3.2 (G)
- net at U4.8 (HB): now also C2.1, D2.1 (K)
- new net: D19.2 (A), R25.1
- new net: TP3.1, U12.4 (AIN0)
- new net: C12.1, R17.2, U12.5 (AIN1)
- new net: C13.1, R9.1, U12.6 (AIN2)
- new net: R12.1, R50.1, U12.7 (AIN3)
- new net: D19.1 (K), Q6.4 (D2)
- new net: D18.1 (K), Q6.5 (D1)
- new net: D2.2 (A), R1.1, R2.1
- new net: D11.2 (A), R11.1
- new net: D12.1 (K), Q1.5 (D1)
- new net: D12.2 (A), R16.1
- new net: D13.2 (A), R18.1
- new net: D9.2 (A), R7.2, U7.2 (G)
- new net: D14.2 (A), R19.1
- new net: D16.2 (A), R21.1, R22.2
- new net: D13.1 (K), Q1.4 (D2)
- new net: D10.1 (K), R8.1, U5.5 (LO)
- new net: D9.1 (K), R7.1, U5.7 (HO)
- new net: C7.1, D8.1 (K), U5.8 (HB)
- new net: C11.1, J4.3 (Pin_3), U6.1 (OUT)
- new net: J5.5 (Pin_5), TP1.1
- new net: D8.2 (A), R5.1, R6.1
- new net: D18.2 (A), R24.1
- new net: D4.1 (K), R3.1, U4.7 (HO)
- new net: J5.6 (Pin_6), TP2.1
- new net: D10.2 (A), R8.2, U8.2 (G)
- new net: D5.2 (A), R4.2, U3.2 (G)
- new net S_Feedback: J5.1 (Pin_1), R9.2
- new net S_Front: J5.2 (Pin_2), R17.1
- new net XDS_3v_supply: J3.3 (Pin_3), J4.1 (Pin_1)
- new net XDS_5v_supply: J3.2 (Pin_2)
- no-connect marks 0 -> 7
Other:
- moved on the sheet: C1, C11, C14, D1, D3, J1, Q2, U1, U2, U3, U4, U6

Commit message: asd
Parts:
- removed J4: Conn_01x03_Pin, Connector_PinHeader_2.54mm:PinHeader_1x03_P2.54mm_Vertical, symbol Connector:Conn_01x03_Pin
- removed Q2: BC846, Package_TO_SOT_SMD:SOT-23, symbol Transistor_BJT:BC846
- removed R1, R5: 8.2, Resistor_SMD:R_2816_7142Metric_Pad3.20x4.45mm_HandSolder, symbol Device:R_Small_US
- removed R18, R24, R25: 750, Resistor_SMD:R_1206_3216Metric_Pad1.30x1.75mm_HandSolder, symbol Device:R_US
- removed R22: 4.99k, Resistor_SMD:R_1206_3216Metric_Pad1.30x1.75mm_HandSolder, symbol Device:R_US
- added J2, J4: Conn_01x02_Pin, Connector_PinHeader_2.54mm:PinHeader_1x02_P2.54mm_Vertical, symbol Connector:Conn_01x02_Pin
- added R1, R5: 49.9k, Resistor_SMD:R_1206_3216Metric_Pad1.30x1.75mm_HandSolder, symbol Device:R_US
- added R13: 2.49k, Resistor_SMD:R_0603_1608Metric, symbol Device:R_US
- added U11: FCX495, Package_TO_SOT_SMD:SOT-89-3, symbol zzLocalLibrary:FCX485_NPN_BJT
- C2, C7: footprint Capacitor_THT:C_Radial_D6.3mm_H11.0mm_P2.50mm -> Capacitor_THT:CP_Radial_D6.3mm_P2.50mm
- J1: footprint Connector_Wago:Wago_734-134_1x04_P3.50mm_Vertical -> Connector_Wire:SolderWire-0.75sqmm_1x04_P4.8mm_D1.25mm_OD2.3mm
- R16: value 750 -> 2.49k; footprint Resistor_SMD:R_1206_3216Metric_Pad1.30x1.75mm_HandSolder -> Resistor_SMD:R_0603_1608Metric; mouser https://www.mouser.com/ProductDetail/YAGEO/RC1206JR-13750RL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 -> https://www.mouser.com/ProductDetail/TE-Connectivity-Holswo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; specs 750mOhm, 250mW, 5%, 100PPM, 200C, -55C, +155C -> (none); unit x10 0.022 -> .03
- R17, R9: value 150 -> 2.49k; footprint Resistor_SMD:R_1206_3216Metric_Pad1.30x1.75mm_HandSolder -> Resistor_SMD:R_0603_1608Metric; mouser https://www.mouser.com/ProductDetail/YAGEO/AC1206FR-7W150RL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 -> https://www.mouser.com/ProductDetail/TE-Connectivity-Holswo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; specs 150Ohm, 500mW, 1%, 200V, -55C, +155C -> (none); unit x10 0.032 -> .03
- R2, R6: value 8.2 -> 5.1; footprint Resistor_SMD:R_2816_7142Metric_Pad3.20x4.45mm_HandSolder -> Resistor_SMD:R_1206_3216Metric_Pad1.30x1.75mm_HandSolder; mouser https://www.mouser.com/ProductDetail/TE-Connectivity-Holswo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 -> https://www.mouser.com/ProductDetail/KOA-Speer/SG73P2BTTD5R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; specs (none) -> 5.1Ohm, 0.33W, 5%, 200ppm, Anti-pulse
- R21: value 4.99k -> 2.49k; footprint Resistor_SMD:R_1206_3216Metric_Pad1.30x1.75mm_HandSolder -> Resistor_SMD:R_0603_1608Metric; mouser https://www.mouser.com/ProductDetail/SEI-Stackpole/RNCP1206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 -> https://www.mouser.com/ProductDetail/TE-Connectivity-Holswo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; specs 4.99kOhm, 200V, 500mW, 1%, 100PPM, -55C, +155C -> (none); unit x10 0.017 -> .03
- R3, R4, R7, R8: footprint Resistor_SMD:R_2512_6332Metric_Pad1.40x3.35mm_HandSolder -> Resistor_SMD:R_1206_3216Metric_Pad1.30x1.75mm_HandSolder; mouser https://www.mouser.com/ProductDetail/TE-Connectivity-Holswo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 -> https://www.mouser.com/ProductDetail/KOA-Speer/SG73P2BTTD5R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; specs (none) -> 5.1Ohm, 0.33W, 5%, 200ppm, Anti-pulse
Connections:
- net +12V: now also R16.2, R17.2, R9.2, R13.2, U11.3; no longer U2.3 (D), U7.3 (D)
- net +3V3: now also J2.1 (Pin_1), J4.2 (Pin_2); no longer R16.2
- net GND: now also J1.4 (Pin_4); no longer J1.3 (Pin_3)
- net M-: now also J1.3 (Pin_3); no longer J1.1 (Pin_1)
- net S_Feedback: now also R5.2; no longer R9.2
- net S_Front: now also R1.1; no longer R17.1
- net TIMG2_C0: now also U4.3 (LI); no longer U4.2 (HI)
- net TIMG2_C1: now also U4.2 (HI); no longer U4.3 (LI)
- net TIMG4_C0: now also U5.3 (LI); no longer U5.2 (HI)
- net TIMG4_C1: now also U5.2 (HI); no longer U5.3 (LI)
- net XDS_3v_supply: now also J4.1 (Pin_1)
- net at D19.2 (A): now also R9.1
- net at C12.1, U12.5 (AIN1): now also R1.2; no longer R17.2
- net at C13.1, U12.6 (AIN2): now also R5.1; no longer R9.1
- net at C1.1, D1.1 (K), R10.1: now also U11.1
- net at D12.2 (A): now also R17.1; no longer R16.1
- net at D13.2 (A): now also R16.1
- net at D10.1 (K), U5.5 (LO): now also R8.2; no longer R8.1
- net +BATT: now reaches D3.2 (A)
- net +BATT: now also J1.1 (Pin_1), U2.3 (D), U7.3 (D); no longer J1.4 (Pin_4)
- net at C11.1, U6.1 (OUT): now also J2.2 (Pin_2)
- net at D18.2 (A): now also R13.1
- net at D10.2 (A), U8.2 (G): now also R8.1; no longer R8.2
- net at D3.1 (K), R10.2: now also U11.2
- net at D5.1 (K), U4.5 (LO): now also R4.2; no longer R4.1
- net at D5.2 (A), U3.2 (G): now also R4.1; no longer R4.2
Other:
- moved on the sheet: D6, D7, J5, TP1, TP2

Commit message: thanks random guy that slaved away at the lower layout
Connections:
- net +3V3: now also J5.6 (Pin_6); no longer J5.4 (Pin_4)
- net at TP2.1: now also J5.4 (Pin_4); no longer J5.6 (Pin_6)
Other:
- moved on the sheet: TP2
Changed lines of the file:
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@@
 	(wire
 		(pts
-			(xy 44.45 46.99) (xy 29.21 46.99)
-		)
-		(stroke
-			(width 0)
-			(type default)
-		)
-	)
-	(wire
-		(pts
 			(xy 24.13 88.9) (xy 25.4 88.9)
 		)
@@
 	(wire
 		(pts
+			(xy 29.21 52.07) (xy 40.64 52.07)
+		)
+		(stroke
+			(width 0)
+			(type default)
+		)
+	)
+	(wire
+		(pts
 			(xy 147.32 29.21) (xy 149.86 29.21)
 		)
@@
 	)
 	(label "Sensor Bias"
-		(at 29.21 46.99 0)
+		(at 29.21 52.07 0)
 		(effects
 			(font
@@
 	(symbol
 		(lib_id "power:+3V3")
-		(at 44.45 46.99 270)
+		(at 40.64 52.07 270)
 		(unit 1)
 		(exclude_from_sim no)
@@
 		(fields_autoplaced yes)
 		(property "Reference" "#PWR018"
-			(at 40.64 46.99 0)
+			(at 36.83 52.07 0)
 			(effects
 				(font
@@
 		)
 		(property "Value" "+3V3"
-			(at 48.26 46.9899 90)
+			(at 44.45 52.0699 90)
 			(effects
 				(font
@@
 		)
 		(property "Footprint" ""
-			(at 44.45 46.99 0)
+			(at 40.64 52.07 0)
 			(effects
 				(font
@@
 		)
 		(property "Datasheet" ""
-			(at 44.45 46.99 0)
+			(at 40.64 52.07 0)
 			(effects
 				(font
@@
 		)
 		(property "Description" "Power symbol creates a global label with name \"+3V3\""
-			(at 44.45 46.99 0)
+			(at 40.64 52.07 0)
 			(effects
 				(font
@@
 	(symbol
 		(lib_id "Connector:TestPoint")
-		(at 29.21 52.07 270)
+		(at 29.21 46.99 270)
 		(unit 1)
 		(exclude_from_sim no)
@@
 		(dnp no)
 		(property "Reference" "TP2"
-			(at 35.814 52.07 90)
+			(at 35.814 46.99 90)
 			(effects
 				(font
@@
 		)
 		(property "Value" "TestPoint"
-			(at 31.2421 54.61 0)
+			(at 31.2421 49.53 0)
 			(effects
 				(font
@@
 		)
 		(property "Footprint" "TestPoint:TestPoint_Loop_D2.50mm_Drill1.0mm_LowProfile"
-			(at 29.21 57.15 0)
+			(at 29.21 52.07 0)
 			(effects
 				(font
@@
 		)
 		(property "Datasheet" "~"
-			(at 29.21 57.15 0)
+			(at 29.21 52.07 0)
 			(effects
 				(font
@@
 		)
 		(property "Description" "test point"
-			(at 29.21 52.07 0)
+			(at 29.21 46.99 0)
 			(effects
 				(font
@@
 		)
 		(property "Sim.Device" ""
-			(at 29.21 52.07 0)
+			(at 29.21 46.99 0)
 			(effects
 				(font
@@
 		)
 		(property "Sim.Type" ""
-			(at 29.21 52.07 0)
+			(at 29.21 46.99 0)
 			(effects
 				(font

Commit message: asd
Parts:
- added R18: 4.99k, Resistor_SMD:R_1206_3216Metric_Pad1.30x1.75mm_HandSolder, symbol Device:R_US
Connections:
- net +3V3: now also R18.1; no longer J5.6 (Pin_6)
- new net Sensor Bias: J5.6 (Pin_6), R18.2
Changed lines of the file:
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@@
 	(wire
 		(pts
+			(xy 40.64 52.07) (xy 44.45 52.07)
+		)
+		(stroke
+			(width 0)
+			(type default)
+		)
+	)
+	(wire
+		(pts
 			(xy 46.99 76.2) (xy 50.8 76.2)
 		)
@@
 	(wire
 		(pts
-			(xy 29.21 52.07) (xy 40.64 52.07)
+			(xy 29.21 52.07) (xy 33.02 52.07)
 		)
 		(stroke
@@
 	)
 	(symbol
+		(lib_id "Device:R_US")
+		(at 36.83 52.07 270)
+		(unit 1)
+		(exclude_from_sim no)
+		(in_bom yes)
+		(on_board yes)
+		(dnp no)
+		(property "Reference" "R18"
+			(at 33.909 54.991 90)
+			(effects
+				(font
+					(size 1.27 1.27)
+				)
+				(justify left)
+			)
+		)
+		(property "Value" "4.99k"
+			(at 33.909 57.531 90)
+			(effects
+				(font
+					(size 1.27 1.27)
+				)
+				(justify left)
+			)
+		)
+		(property "Footprint" "Resistor_SMD:R_1206_3216Metric_Pad1.30x1.75mm_HandSolder"
+			(at 36.576 53.086 90)
+			(effects
+				(font
+					(size 1.27 1.27)
+				)
+				(hide yes)
+			)
+		)
+		(property "Datasheet" ""
+			(at 36.83 52.07 0)
+			(effects
+				(font
+					(size 1.27 1.27)
+				)
+				(hide yes)
+			)
+		)
+		(property "Description" "Resistor, US symbol"
+			(at 36.83 52.07 0)
+			(effects
+				(font
+					(size 1.27 1.27)
+				)
+				(hide yes)
+			)
+		)
+		(property "Sim.Device" ""
+			(at 36.83 52.07 90)
+			(effects
+				(font
+					(size 1.27 1.27)
+				)
+				(hide yes)
+			)
+		)
+		(property "Sim.Type" ""
+			(at 36.83 52.07 90)
+			(effects
+				(font
+					(size 1.27 1.27)
+				)
+				(hide yes)
+			)
+		)
+		(property "mouser" "https://www.mouser.com/ProductDetail/SEI-Stackpole/RNCP1206FTD4K99?qs=sGAEpiMZZMvdGkrng054tyMPH50YnZ95yR%2FF2bQQIaAb5UdPiGbTtQ%3D%3D"
+			(at 36.83 52.07 0)
+			(effects
+				(font
+					(size 1.27 1.27)
+				)
+				(hide yes)
+			)
+		)
+		(property "specs" "4.99kOhm, 200V, 500mW, 1%, 100PPM, -55C, +155C"
+			(at 36.83 52.07 0)
+			(effects
+				(font
+					(size 1.27 1.27)
+				)
+				(hide yes)
+			)
+		)
+		(property "unit x10" "0.017"
+			(at 36.83 52.07 0)
+			(effects
+				(font
+					(size 1.27 1.27)
+				)
+				(hide yes)
+			)
+		)
+		(pin "1"
+		)
+		(pin "2"
+		)
+		(instances
+			(project "FWS_20A"
+				(path "/bd07da4b-c018-42fa-9039-1b3b7c5adf19"
+					(reference "R18")
+					(unit 1)
+				)
+			)
+		)
+	)
+	(symbol
 		(lib_id "Regulator_Linear:L78L33_SO8")
 		(at 119.38 29.21 0)
@@
 	(symbol
 		(lib_id "power:+3V3")
-		(at 40.64 52.07 270)
+		(at 44.45 52.07 270)
 		(unit 1)
 		(exclude_from_sim no)
@@
 		(fields_autoplaced yes)
 		(property "Reference" "#PWR018"
-			(at 36.83 52.07 0)
+			(at 40.64 52.07 0)
 			(effects
 				(font
@@
 		)
 		(property "Value" "+3V3"
-			(at 44.45 52.0699 90)
+			(at 48.26 52.0699 90)
 			(effects
 				(font
@@
 		)
 		(property "Footprint" ""
-			(at 40.64 52.07 0)
+			(at 44.45 52.07 0)
 			(effects
 				(font
@@
 		)
 		(property "Datasheet" ""
-			(at 40.64 52.07 0)
+			(at 44.45 52.07 0)
 			(effects
 				(font
@@
 		)
 		(property "Description" "Power symbol creates a global label with name \"+3V3\""
-			(at 40.64 52.07 0)
+			(at 44.45 52.07 0)
 			(effects
 				(font

Commit message: sad
Parts:
- added TP4, TP5: TestPoint, TestPoint:TestPoint_Pad_D2.0mm, symbol Connector:TestPoint
Connections:
- net I2C0_SCL: now also TP4.1
- net I2C0_SDA: now also TP5.1
Changed lines of the file:
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@@
 	(wire
 		(pts
+			(xy 134.62 91.44) (xy 134.62 97.79)
+		)
+		(stroke
+			(width 0)
+			(type default)
+		)
+	)
+	(wire
+		(pts
 			(xy 134.62 91.44) (xy 168.91 91.44)
 		)
@@
 	(wire
 		(pts
+			(xy 138.43 93.98) (xy 138.43 97.79)
+		)
+		(stroke
+			(width 0)
+			(type default)
+		)
+	)
+	(wire
+		(pts
 			(xy 95.25 81.28) (xy 95.25 83.82)
 		)
@@
 	)
 	(symbol
+		(lib_id "Connector:TestPoint")
+		(at 138.43 97.79 180)
+		(unit 1)
+		(exclude_from_sim no)
+		(in_bom no)
+		(on_board yes)
+		(dnp no)
+		(property "Reference" "TP5"
+			(at 138.43 104.394 90)
+			(effects
+				(font
+					(size 1.27 1.27)
+				)
+			)
+		)
+		(property "Value" "TestPoint"
+			(at 135.89 99.8221 0)
+			(effects
+				(font
+					(size 1.27 1.27)
+				)
+				(justify left)
+				(hide yes)
+			)
+		)
+		(property "Footprint" "TestPoint:TestPoint_Pad_D2.0mm"
+			(at 133.35 97.79 0)
+			(effects
+				(font
+					(size 1.27 1.27)
+				)
+				(hide yes)
+			)
+		)
+		(property "Datasheet" "~"
+			(at 133.35 97.79 0)
+			(effects
+				(font
+					(size 1.27 1.27)
+				)
+				(hide yes)
+			)
+		)
+		(property "Description" "test point"
+			(at 138.43 97.79 0)
+			(effects
+				(font
+					(size 1.27 1.27)
+				)
+				(hide yes)
+			)
+		)
+		(property "Sim.Device" ""
+			(at 138.43 97.79 0)
+			(effects
+				(font
+					(size 1.27 1.27)
+				)
+				(hide yes)
+			)
+		)
+		(property "Sim.Type" ""
+			(at 138.43 97.79 0)
+			(effects
+				(font
+					(size 1.27 1.27)
+				)
+				(hide yes)
+			)
+		)
+		(pin "1"
+		)
+		(instances
+			(project "FWS_20A"
+				(path "/bd07da4b-c018-42fa-9039-1b3b7c5adf19"
+					(reference "TP5")
+					(unit 1)
+				)
+			)
+		)
+	)
+	(symbol
 		(lib_id "power:+12V")
 		(at 250.19 158.75 90)
@@
 					(unit 1)
 				)
+			)
+		)
+	)
+	(symbol
+		(lib_id "Connector:TestPoint")
+		(at 134.62 97.79 180)
+		(unit 1)
+		(exclude_from_sim no)
+		(in_bom no)
+		(on_board yes)
+		(dnp no)
+		(property "Reference" "TP4"
+			(at 134.62 104.394 90)
+			(effects
+				(font
+					(size 1.27 1.27)
+				)
+			)
+		)
+		(property "Value" "TestPoint"
+			(at 132.08 99.8221 0)
+			(effects
+				(font
+					(size 1.27 1.27)
+				)
+				(justify left)
+				(hide yes)
+			)
+		)
+		(property "Footprint" "TestPoint:TestPoint_Pad_D2.0mm"
+			(at 129.54 97.79 0)
+			(effects
+				(font
+					(size 1.27 1.27)
+				)
+				(hide yes)
+			)
+		)
+		(property "Datasheet" "~"
+			(at 129.54 97.79 0)
+			(effects
+				(font
+					(size 1.27 1.27)
+				)
+				(hide yes)
+			)
+		)
+		(property "Description" "test point"
+			(at 134.62 97.79 0)
+			(effects
+				(font
+					(size 1.27 1.27)
+				)
+				(hide yes)
+			)
+		)
+		(property "Sim.Device" ""
+			(at 134.62 97.79 0)
+			(effects
+				(font
+					(size 1.27 1.27)
+				)
+				(hide yes)
+			)
+		)
+		(property "Sim.Type" ""
+			(at 134.62 97.79 0)
+			(effects
+				(font
+					(size 1.27 1.27)
+				)
+				(hide yes)
+			)
+		)
+		(pin "1"
+		)
+		(instances
+			(project "FWS_20A"
+				(path "/bd07da4b-c018-42fa-9039-1b3b7c5adf19"
+					(reference "TP4")
+					(unit 1)
+				)

Commit message: cleaned a bit
Parts:
- added D15, D17: 3.3V, Diode_SMD:D_SOD-323, symbol Device:D_Zener
- added TP6, TP7, TP8, TP9: TestPoint, TestPoint:TestPoint_Pad_D2.0mm, symbol Connector:TestPoint
Connections:
- net GND: now also D15.2 (A), D17.2 (A)
- net TIMG2_C0: now also TP7.1
- net TIMG2_C1: now also TP6.1
- net TIMG4_C0: now also TP8.1
- net TIMG4_C1: now also TP9.1
- net at C12.1, R1.2, U12.5 (AIN1): now also D15.1 (K)
- net at C13.1, R5.1, U12.6 (AIN2): now also D17.1 (K)
Other:
- moved on the sheet: C12, C13
